File: board-v6/NyanTimer-v6.brd (EAGLE design)
At the start: 136.3 x 45 mm, 46 parts, among them IC1 7815DT, IC2 MAX232, IC3 7815DT, SW1 AKIZUKI_SWITCH, U1 328P

Commit message: modified board
Parts:
- moved SW1 0.10 mm to (14.0, 42.9)
Routing:
- net GND: track 298.7 -> 0.00 mm, vias 2 -> 0
- net SCL: track 83.0 -> 110.8 mm
- net LEDR: track 40.7 -> 68.4 mm, vias 0 -> 2
- net LEDG: track 66.0 -> 43.4 mm, vias 2 -> 1
- net PADRIN: track 111.4 -> 94.9 mm, vias 1 -> 4
- net SDA: track 101.1 -> 90.6 mm, vias 4 -> 2
- net SW2: track 75.9 -> 85.4 mm
- net VCC: track 208.4 -> 199.9 mm
- net SW3: track 86.3 -> 78.0 mm, vias 1 -> 2
- net PHONE: track 64.8 -> 57.2 mm
- net BUZ+: track 52.5 -> 58.0 mm, vias 0 -> 3
- net PADR: track 98.2 -> 103.7 mm, vias 0 -> 3
- net SW4: track 48.9 -> 53.9 mm
- net SW1: track 72.5 -> 67.7 mm, vias 0 -> 2
- net T2IN: track 43.0 -> 47.7 mm, vias 0 -> 1
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
Commit message: modified board
Routing:
- net GND: track 0.00 -> 309.2 mm, vias 0 -> 4
- net LEDG: track 43.4 -> 63.4 mm, vias 1 -> 2
- net PADRIN: track 94.9 -> 113.6 mm, vias 4 -> 3
- net +5V: track 132.7 -> 151.0 mm
- net SCL: track 110.8 -> 93.5 mm
- net VCC: track 199.9 -> 182.7 mm
- net SW1: track 67.7 -> 82.4 mm
- net LEDR: track 68.4 -> 54.5 mm, vias 2 -> 0
- net N$2: track 15.9 -> 27.5 mm, vias 1 -> 0
- net SDA: track 90.6 -> 80.6 mm, vias 2 -> 3
- net VSWOUT: track 26.5 -> 35.2 mm, vias 2 -> 1
- net SW3: track 78.0 -> 70.0 mm, vias 2 -> 3
- net PHONE: track 57.2 -> 64.8 mm
- net SW2: track 85.4 -> 78.3 mm, vias 1 -> 3
- net VSW: track 94.7 -> 89.3 mm
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