File: board/board-v7/NyanTimer-v7.brd (EAGLE design)
At the start: 136 x 45 mm, 49 parts, among them IC1 7815DT, IC2 MAX232, IC3 7815DT, SW1 AKIZUKI_SWITCH, U1 328P

Commit message: modified
Parts:
- moved C3 1.41 mm to (31.1, 18.3), turned to 180 degrees
Changed lines of the file:
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@@
 </layers>
 <board>
+<fusionsync huburn="a.cGVyc29uYWw6dWUyZDY1ODA3" projecturn="a.cGVyc29uYWw6dWUyZDY1ODA3IzIwMTgwOTMwMTUxNjc4Mzgx" f3durn="urn:adsk.wipprod:dm.lineage:HZn5fMgTTJKOyip3mBVZMA" pcbguid="90678893-8f50-44b1-a255-14d25019db93" lastpulledtime="" lastsyncedchangeguid="f16c29d8-f572-6caa-3653-47bf9a888ec9"/>
 <plain>
 <hole x="-42" y="4" drill="3"/>
@@
 <attribute name="VALUE" x="31.473" y="7.388" size="1.27" layer="27" ratio="10" rot="R270"/>
 </element>
-<element name="C3" library="rcl" library_urn="urn:adsk.eagle:library:334" package="C025-024X044" package3d_urn="urn:adsk.eagle:package:23630/1" value="0.1u" x="30.14" y="19.28" smashed="yes" rot="R90">
-<attribute name="NAME" x="32.743" y="21.502" size="1.27" layer="25" ratio="10" rot="R90"/>
-<attribute name="POPULARITY" value="56" x="30.14" y="19.28" size="1.778" layer="27" rot="R90" display="off"/>
-<attribute name="SPICEPREFIX" value="C" x="91.1" y="39.6" size="1.778" layer="27" rot="R90" display="off"/>
-<attribute name="VALUE" x="32.807" y="17.502" size="1.27" layer="27" ratio="10" rot="R90"/>
+<element name="C3" library="rcl" library_urn="urn:adsk.eagle:library:334" package="C025-024X044" package3d_urn="urn:adsk.eagle:package:23630/1" value="0.1u" x="31.14" y="18.28" smashed="yes" rot="R180">
+<attribute name="NAME" x="28.918" y="20.883" size="1.27" layer="25" ratio="10" rot="R180"/>
+<attribute name="POPULARITY" value="56" x="31.14" y="18.28" size="1.778" layer="27" rot="R180" display="off"/>
+<attribute name="SPICEPREFIX" value="C" x="10.82" y="79.24" size="1.778" layer="27" rot="R180" display="off"/>
+<attribute name="VALUE" x="32.918" y="20.947" size="1.27" layer="27" ratio="10" rot="R180"/>
 </element>
 <element name="C4" library="rcl" library_urn="urn:adsk.eagle:library:334" package="C025-024X044" package3d_urn="urn:adsk.eagle:package:23630/1" value="0.1u" x="-34.16" y="11.2" smashed="yes" rot="R90">
@@
 <contactref element="C9" pad="1"/>
 <contactref element="C10" pad="1"/>
-<wire x1="22.78" y1="27.04" x2="30.14" y2="18.01" width="0" layer="19" extent="1-1"/>
+<wire x1="22.78" y1="27.04" x2="32.41" y2="18.28" width="0" layer="19" extent="1-1"/>
 <wire x1="22.8" y1="18.04" x2="22.78" y2="27.04" width="0" layer="19" extent="1-1"/>
 <wire x1="34.14" y1="6.88" x2="22.8" y2="18.04" width="0" layer="19" extent="1-1"/>
@@
 <contactref element="U1" pad="13"/>
 <contactref element="CONNECTOR3" pad="4"/>
-<wire x1="27.28" y1="27.04" x2="30.14" y2="20.55" width="0" layer="19" extent="1-1"/>
+<wire x1="27.28" y1="27.04" x2="29.87" y2="18.28" width="0" layer="19" extent="1-1"/>
 <wire x1="6.37" y1="11.2" x2="27.28" y2="27.04" width="0" layer="19" extent="1-1"/>
 <wire x1="-5.05" y1="35.28" x2="6.37" y2="11.2" width="0" layer="19" extent="1-1"/>
@@
 </note>
 <note version="8.3" severity="warning">
+Since Version 8.3, EAGLE supports Fusion synchronisation.
+This feature will not be available in this version and saving
+the document will break the link to the Fusion PCB feature.
+</note>
+<note version="8.3" severity="warning">

Commit message: routed
Routing:
- net GND: track 0.00 -> 266.8 mm, vias 0 -> 2
- net VCC: track 0.00 -> 194.0 mm, vias 0 -> 1
- net +5V: track 0.00 -> 187.9 mm, vias 0 -> 1
- net T2IN: track 0.00 -> 139.9 mm, vias 0 -> 8
- net N$7: track 0.00 -> 138.1 mm, vias 0 -> 3
- net VSW: track 0.00 -> 121.3 mm, vias 0 -> 3
- net SCL: track 0.00 -> 108.1 mm, vias 0 -> 1
- net PADRIN: track 0.00 -> 107.4 mm, vias 0 -> 3
- net BUZ+: track 0.00 -> 93.4 mm, vias 0 -> 4
- net LEDG: track 0.00 -> 86.7 mm, vias 0 -> 2
- net SDA: track 0.00 -> 85.9 mm, vias 0 -> 2
- net SW3: track 0.00 -> 84.7 mm, vias 0 -> 2
- net SW2: track 0.00 -> 78.3 mm
- net PHONE: track 0.00 -> 74.3 mm, vias 0 -> 2
- net PADR: track 0.00 -> 70.6 mm
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
Commit message: routed
Routing:
- net GND: track 266.8 -> 0.00 mm, vias 2 -> 0
- net N$7: track 138.1 -> 93.6 mm, vias 3 -> 0
- net BUZ+: track 93.4 -> 59.5 mm, vias 4 -> 3
- net LEDG: track 86.7 -> 54.7 mm
- net PADR: track 70.6 -> 97.0 mm, vias 0 -> 1
- net VSW: track 121.3 -> 98.4 mm
- net SCL: track 108.1 -> 88.2 mm
- net PADRIN: track 107.4 -> 88.0 mm, vias 3 -> 1
- net N$12: track 14.5 -> 33.2 mm, vias 1 -> 0
- net SW3: track 84.7 -> 67.0 mm
- net T2IN: track 139.9 -> 125.2 mm, vias 8 -> 1
- net +5V: track 187.9 -> 201.8 mm, vias 1 -> 3
- net N$11: track 27.2 -> 14.0 mm, vias 1 -> 0
- net LEDR: track 56.3 -> 46.7 mm
- net SDA: track 85.9 -> 77.6 mm, vias 2 -> 1
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- added copper zone on layer 1, net GND
- added copper zone on layer 16, net GND

Commit message: routed
Routing:
- net GND: track 0.00 -> 289.8 mm, vias 0 -> 6
- net N$7: track 93.6 -> 138.1 mm, vias 0 -> 3
- net BUZ+: track 59.5 -> 93.4 mm, vias 3 -> 4
- net LEDG: track 54.7 -> 86.7 mm
- net PADR: track 97.0 -> 70.6 mm, vias 1 -> 0
- net VSW: track 98.4 -> 121.3 mm
- net SCL: track 88.2 -> 108.1 mm
- net PADRIN: track 88.0 -> 107.4 mm, vias 1 -> 3
- net N$12: track 33.2 -> 14.5 mm, vias 0 -> 1
- net SW3: track 67.0 -> 84.7 mm
- net T2IN: track 125.2 -> 139.9 mm, vias 1 -> 8
- net +5V: track 201.8 -> 187.9 mm, vias 3 -> 1
- net N$11: track 14.0 -> 27.2 mm, vias 0 -> 1
- net LEDR: track 46.7 -> 56.3 mm
- net SDA: track 77.6 -> 85.9 mm, vias 1 -> 2
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