File: board/board-v7/NyanTimer-v7.brd (EAGLE design)
At the start: 136 x 45 mm, 50 parts, among them IC1 7815DT, IC2 MAX232, IC3 7815DT, SW1 AKIZUKI_SWITCH, U1 328P

Commit message: modified
Parts:
- moved BT1 1.50 mm to (-33.6, 24.2)
- moved BT2 1.50 mm to (33.6, 24.2)
- moved SV1 0.50 mm to (-44.0, 40.5)
Changed lines of the file:
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@@
 <setting verticaltext="up"/>
 </settings>
-<grid distance="4" unitdist="mm" unit="mm" style="lines" multiple="1" display="yes" altdistance="0.25" altunitdist="mm" altunit="mm"/>
+<grid distance="1" unitdist="mm" unit="mm" style="lines" multiple="1" display="yes" altdistance="0.25" altunitdist="mm" altunit="mm"/>
 <layers>
 <layer number="1" name="Top" color="4" fill="1" visible="yes" active="yes"/>
@@
 <attribute name="VALUE" x="7.612" y="24.003" size="1.27" layer="27" ratio="10"/>
 </element>
-<element name="BT1" library="akizuki_cr2032" package="AKIZUKI_CR2032" value="AKIZUKI_CR2032" x="-33.65" y="25.75" smashed="yes" rot="R90"/>
-<element name="BT2" library="akizuki_cr2032" package="AKIZUKI_CR2032" value="AKIZUKI_CR2032" x="33.65" y="25.75" smashed="yes" rot="SR270"/>
+<element name="BT1" library="akizuki_cr2032" package="AKIZUKI_CR2032" value="AKIZUKI_CR2032" x="-33.65" y="24.25" smashed="yes" rot="R90"/>
+<element name="BT2" library="akizuki_cr2032" package="AKIZUKI_CR2032" value="AKIZUKI_CR2032" x="33.65" y="24.25" smashed="yes" rot="SR270"/>
 <element name="R9" library="resistor" library_urn="urn:adsk.eagle:library:348" package="0207/10" package3d_urn="urn:adsk.eagle:package:23491/2" value="10k" x="-29.45" y="31.75" smashed="yes" rot="R180">
 <attribute name="NAME" x="-26.402" y="30.226" size="1.27" layer="25" ratio="10" rot="R180"/>
@@
 <attribute name="VALUE" x="1.167" y="27.422" size="1.27" layer="27" ratio="10" rot="R90"/>
 </element>
-<element name="SV1" library="con-lstb" library_urn="urn:adsk.eagle:library:162" package="MA06-1" package3d_urn="urn:adsk.eagle:package:8340/1" value="" x="-44" y="41" smashed="yes">
-<attribute name="MF" value="" x="-44" y="41" size="1.778" layer="27" display="off"/>
-<attribute name="MPN" value="" x="-44" y="41" size="1.778" layer="27" display="off"/>
-<attribute name="NAME" x="-51.62" y="42.651" size="1.27" layer="25" ratio="10"/>
-<attribute name="OC_FARNELL" value="unknown" x="-44" y="41" size="1.778" layer="27" display="off"/>
-<attribute name="OC_NEWARK" value="unknown" x="-44" y="41" size="1.778" layer="27" display="off"/>
-<attribute name="POPULARITY" value="28" x="-44" y="41" size="1.778" layer="27" display="off"/>
-<attribute name="VALUE" x="-46.54" y="38.079" size="1.27" layer="27" ratio="10"/>
+<element name="SV1" library="con-lstb" library_urn="urn:adsk.eagle:library:162" package="MA06-1" package3d_urn="urn:adsk.eagle:package:8340/1" value="" x="-44" y="40.5" smashed="yes">
+<attribute name="MF" value="" x="-44" y="40.5" size="1.778" layer="27" display="off"/>
+<attribute name="MPN" value="" x="-44" y="40.5" size="1.778" layer="27" display="off"/>
+<attribute name="NAME" x="-51.62" y="42.151" size="1.27" layer="25" ratio="10"/>
+<attribute name="OC_FARNELL" value="unknown" x="-44" y="40.5" size="1.778" layer="27" display="off"/>
+<attribute name="OC_NEWARK" value="unknown" x="-44" y="40.5" size="1.778" layer="27" display="off"/>
+<attribute name="POPULARITY" value="28" x="-44" y="40.5" size="1.778" layer="27" display="off"/>
+<attribute name="VALUE" x="-46.54" y="37.579" size="1.27" layer="27" ratio="10"/>
 </element>
 </elements>
@@
 <contactref element="C18" pad="2"/>
 <contactref element="SV1" pad="1"/>
-<wire x1="53.97" y1="25.75" x2="63.3" y2="27.12" width="0" layer="19" extent="1-1"/>
+<wire x1="53.97" y1="24.25" x2="63.3" y2="27.12" width="0" layer="19" extent="1-1"/>
 <wire x1="69.13" y1="17.15" x2="63.3" y2="27.12" width="0" layer="19" extent="1-1"/>
 <wire x1="65.79" y1="13.14" x2="69.13" y2="17.15" width="0" layer="19" extent="1-1"/>
-<wire x1="32.22" y1="37.16" x2="53.97" y2="25.75" width="0" layer="19" extent="1-1"/>
+<wire x1="32.22" y1="37.16" x2="53.97" y2="24.25" width="0" layer="19" extent="1-1"/>
 <wire x1="17.74" y1="35.56" x2="32.22" y2="37.16" width="0" layer="19" extent="1-1"/>
 <wire x1="18.25" y1="28.91" x2="17.74" y2="35.56" width="0" layer="19" extent="1-1"/>
@@
 <wire x1="-18.17" y1="29.03" x2="-19.82" y2="31.75" width="0" layer="19" extent="1-1"/>
 <wire x1="-18.29" y1="42.9" x2="-15.75" y2="35.28" width="0" layer="19" extent="1-1"/>
-<wire x1="-50.35" y1="41" x2="-19.82" y2="31.75" width="0" layer="19" extent="1-1"/>
+<wire x1="-50.35" y1="40.5" x2="-19.82" y2="31.75" width="0" layer="19" extent="1-1"/>
 </signal>
 <signal name="+5V">
@@
 <wire x1="-34.16" y1="9.93" x2="-27.27" y2="17.98" width="0" layer="19" extent="1-1"/>
 <wire x1="-34.18" y1="4.34" x2="-34.16" y2="9.93" width="0" layer="19" extent="1-1"/>
-<wire x1="-45.27" y1="41" x2="-27.24" y2="27.04" width="0" layer="19" extent="1-1"/>
+<wire x1="-45.27" y1="40.5" x2="-27.24" y2="27.04" width="0" layer="19" extent="1-1"/>
 </signal>
 <signal name="BUZ+">
@@
 <contactref element="SW1" pad="PIN1"/>
 <contactref element="BT1" pad="PLUS"/>
-<wire x1="-33.65" y1="25.75" x2="16" y2="42.9" width="0" layer="19" extent="1-1"/>
+<wire x1="-33.65" y1="24.25" x2="16" y2="42.9" width="0" layer="19" extent="1-1"/>
 </signal>
 <signal name="VSWOUT">
@@
 <contactref element="BT1" pad="MINUS"/>
 <contactref element="BT2" pad="PLUS"/>
-<wire x1="-53.97" y1="25.75" x2="33.65" y2="25.75" width="0" layer="19" extent="1-1"/>
+<wire x1="-53.97" y1="24.25" x2="33.65" y2="24.25" width="0" layer="19" extent="1-1"/>
 </signal>
 <signal name="N$8">

Commit message: routed
Parts:
- added C19: 0.1u, rcl:C025-024X044
- moved SV1 1.00 mm to (-44.0, 41.5)
Connections:
- removed net N$8: R9.2, U1.1
- new net N$6: C19.1, SV1.6
- new net RESET: C19.2, R9.2, U1.1
- new net RX: SV1.4, U1.2
- net GND: now also SV1.2
- net T2IN: now also SV1.5
Routing:
- net GND: track 0.00 -> 278.8 mm, vias 0 -> 1
- net +5V: track 0.00 -> 160.4 mm, vias 0 -> 2
- net VCC: track 0.00 -> 155.5 mm, vias 0 -> 2
- net SCL: track 0.00 -> 125.4 mm, vias 0 -> 1
- net T2IN: track 0.00 -> 124.4 mm, vias 0 -> 3
- net N$7: track 0.00 -> 118.8 mm, vias 0 -> 3
- net PADRIN: track 0.00 -> 95.5 mm, vias 0 -> 4
- net LEDG: track 0.00 -> 90.7 mm, vias 0 -> 1
- net VSW: track 0.00 -> 81.8 mm, vias 0 -> 4
- net SDA: track 0.00 -> 80.4 mm, vias 0 -> 2
- net SW3: track 0.00 -> 78.8 mm, vias 0 -> 1
- net PADR: track 0.00 -> 76.2 mm, vias 0 -> 6
- net SW2: track 0.00 -> 73.8 mm, vias 0 -> 3
- net PHONE: track 0.00 -> 69.9 mm
- net SW4: track 0.00 -> 58.5 mm, vias 0 -> 1
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
Commit message: changed pad
Connections:
- net BUZ+: now also U1.11; no longer U1.23
- net PADLIN: now also U1.23; no longer U1.25
- net PADR: now also U1.25; no longer U1.4
Routing:
- net +5V: track 160.4 -> 214.8 mm, vias 2 -> 1
- net LEDG: track 90.7 -> 40.6 mm, vias 1 -> 2
- net GND: track 278.8 -> 323.7 mm, vias 1 -> 2
- net SW2: track 73.8 -> 117.9 mm, vias 3 -> 2
- net T2IN: track 124.4 -> 159.8 mm
- net N$9: track 11.7 -> 41.7 mm
- net VCC: track 155.5 -> 185.4 mm, vias 2 -> 0
- net N$7: track 118.8 -> 92.8 mm, vias 3 -> 0
- net SCL: track 125.4 -> 104.5 mm, vias 1 -> 2
- net N$14: track 31.6 -> 50.9 mm, vias 0 -> 1
- net VSW: track 81.8 -> 92.5 mm, vias 4 -> 3
- net PHONE: track 69.9 -> 79.8 mm, vias 0 -> 2
- net BUZ+: track 50.4 -> 41.0 mm, vias 2 -> 0
- net PADLIN: track 48.6 -> 57.9 mm, vias 1 -> 2
- net SW3: track 78.8 -> 85.3 mm, vias 1 -> 5
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