File: board/board-v7/NyanTimer-v7.sch (EAGLE design)
At the start: 49 parts, among them IC1 7815DT, IC2 MAX232, IC3 7815DT, SW1 AKIZUKI_SWITCH, U1 328P

Commit message: modified
Parts:
- C11, C9: value 0.1u -> 2.2u
- C8: value 200u -> 0.1u
Changed lines of the file:
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@@
 <part name="GND6" library="supply1" library_urn="urn:adsk.eagle:library:371" deviceset="GND" device=""/>
 <part name="SW1" library="akizuki_switch" deviceset="AKIZUKI_SWITCH" device=""/>
-<part name="C8" library="rcl" library_urn="urn:adsk.eagle:library:334" deviceset="C-EU" device="025-024X044" package3d_urn="urn:adsk.eagle:package:23630/1" value="200u"/>
-<part name="C9" library="rcl" library_urn="urn:adsk.eagle:library:334" deviceset="C-EU" device="025-024X044" package3d_urn="urn:adsk.eagle:package:23630/1" value="0.1u"/>
+<part name="C8" library="rcl" library_urn="urn:adsk.eagle:library:334" deviceset="C-EU" device="025-024X044" package3d_urn="urn:adsk.eagle:package:23630/1" value="0.1u"/>
+<part name="C9" library="rcl" library_urn="urn:adsk.eagle:library:334" deviceset="C-EU" device="025-024X044" package3d_urn="urn:adsk.eagle:package:23630/1" value="2.2u"/>
 <part name="BT1" library="akizuki_cr2032" deviceset="AKIZUKI_CR2032" device=""/>
 <part name="BT2" library="akizuki_cr2032" deviceset="AKIZUKI_CR2032" device=""/>
@@
 <part name="IC3" library="linear" library_urn="urn:adsk.eagle:library:262" deviceset="78*" device="DT" package3d_urn="urn:adsk.eagle:package:16415/2" technology="15"/>
 <part name="GND16" library="supply1" library_urn="urn:adsk.eagle:library:371" deviceset="GND" device=""/>
-<part name="C11" library="rcl" library_urn="urn:adsk.eagle:library:334" deviceset="C-EU" device="025-024X044" package3d_urn="urn:adsk.eagle:package:23630/1" value="0.1u"/>
+<part name="C11" library="rcl" library_urn="urn:adsk.eagle:library:334" deviceset="C-EU" device="025-024X044" package3d_urn="urn:adsk.eagle:package:23630/1" value="2.2u"/>
 <part name="C12" library="rcl" library_urn="urn:adsk.eagle:library:334" deviceset="C-EU" device="025-024X044" package3d_urn="urn:adsk.eagle:package:23630/1" value="0.1u"/>
 <part name="C13" library="rcl" library_urn="urn:adsk.eagle:library:334" deviceset="C-EU" device="025-024X044" package3d_urn="urn:adsk.eagle:package:23630/1" value="0.1u"/>

Commit message: modified padl pin
Connections:
- net PADLIN: now also U1.PC2(ADC2); no longer U1.PD5(T1)
Changed lines of the file:
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@@
 </segment>
 <segment>
-<pinref part="U1" gate="G$1" pin="PD5(T1)"/>
-<wire x1="57.15" y1="106.68" x2="58.42" y2="106.68" width="0.1524" layer="91"/>
-<label x="58.42" y="106.68" size="1.778" layer="95"/>
+<pinref part="U1" gate="G$1" pin="PC2(ADC2)"/>
+<wire x1="57.15" y1="137.16" x2="58.42" y2="137.16" width="0.1524" layer="91"/>
+<label x="58.42" y="137.16" size="1.778" layer="95"/>
 </segment>
 </net>

Commit message: mounted USB-Serial pinhead
Parts:
- added SV1: (no value), con-lstb:MA06-1
Changed lines of the file:
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@@
 <part name="C17" library="rcl" library_urn="urn:adsk.eagle:library:334" deviceset="C-EU" device="025-024X044" package3d_urn="urn:adsk.eagle:package:23630/1" value="22p"/>
 <part name="C18" library="rcl" library_urn="urn:adsk.eagle:library:334" deviceset="C-EU" device="025-024X044" package3d_urn="urn:adsk.eagle:package:23630/1" value="22p"/>
+<part name="SV1" library="con-lstb" library_urn="urn:adsk.eagle:library:162" deviceset="MA06-1" device="" package3d_urn="urn:adsk.eagle:package:8340/1"/>
 </parts>
 <sheets>
@@
 <attribute name="VALUE" x="86.614" y="165.481" size="1.778" layer="96"/>
 </instance>
+<instance part="SV1" gate="1" x="54.61" y="20.32" smashed="yes">
+<attribute name="VALUE" x="53.34" y="7.62" size="1.778" layer="96"/>
+<attribute name="NAME" x="53.34" y="28.702" size="1.778" layer="95"/>
+</instance>
 </instances>

Commit message: modified
Connections:
- net GND: now also SV1.1
Changed lines of the file:
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@@
 <wire x1="-5.08" y1="96.52" x2="-5.08" y2="95.25" width="0.1524" layer="91"/>
+</segment>
+<segment>
+<pinref part="SV1" gate="1" pin="1"/>
+<wire x1="62.23" y1="12.7" x2="64.77" y2="12.7" width="0.1524" layer="91"/>
+<label x="64.77" y="12.7" size="1.778" layer="95"/>
 </segment>
 </net>

Commit message: modified
Connections:
- net +5V: now also SV1.3
Changed lines of the file:
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@@
 <part name="C18" library="rcl" library_urn="urn:adsk.eagle:library:334" deviceset="C-EU" device="025-024X044" package3d_urn="urn:adsk.eagle:package:23630/1" value="22p"/>
 <part name="SV1" library="con-lstb" library_urn="urn:adsk.eagle:library:162" deviceset="MA06-1" device="" package3d_urn="urn:adsk.eagle:package:8340/1"/>
+<part name="P+8" library="supply1" library_urn="urn:adsk.eagle:library:371" deviceset="+5V" device=""/>
+<part name="GND14" library="supply1" library_urn="urn:adsk.eagle:library:371" deviceset="GND" device=""/>
 </parts>
 <sheets>
@@
 <attribute name="VALUE" x="53.34" y="7.62" size="1.778" layer="96"/>
 <attribute name="NAME" x="53.34" y="28.702" size="1.778" layer="95"/>
+</instance>
+<instance part="P+8" gate="1" x="64.77" y="17.78" smashed="yes" rot="R270">
+<attribute name="VALUE" x="59.69" y="20.32" size="1.778" layer="96"/>
+</instance>
+<instance part="GND14" gate="1" x="64.77" y="12.7" smashed="yes" rot="R90">
+<attribute name="VALUE" x="67.31" y="10.16" size="1.778" layer="96" rot="R90"/>
 </instance>
 </instances>
@@
 </segment>
 <segment>
+<pinref part="GND14" gate="1" pin="GND"/>
 <pinref part="SV1" gate="1" pin="1"/>
-<wire x1="62.23" y1="12.7" x2="64.77" y2="12.7" width="0.1524" layer="91"/>
-<label x="64.77" y="12.7" size="1.778" layer="95"/>
 </segment>
 </net>
@@
 <wire x1="-5.08" y1="107.95" x2="-5.08" y2="104.14" width="0.1524" layer="91"/>
 </segment>
+<segment>
+<pinref part="P+8" gate="1" pin="+5V"/>
+<pinref part="SV1" gate="1" pin="3"/>
+</segment>
 </net>

Commit message: routed
Parts:
- added C19: 0.1u, rcl:C-EU025-024X044
Connections:
- removed net N$8: R9.2, U1.PC6(/RESET)
- new net N$6: C19.1, SV1.6
- new net RESET: C19.2, R9.2, U1.PC6(/RESET)
- new net RX: SV1.4, U1.PD0(RXD)
- net GND: now also SV1.2
- net T2IN: now also SV1.5
Changed lines of the file:
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@@
 <part name="P+8" library="supply1" library_urn="urn:adsk.eagle:library:371" deviceset="+5V" device=""/>
 <part name="GND14" library="supply1" library_urn="urn:adsk.eagle:library:371" deviceset="GND" device=""/>
+<part name="GND19" library="supply1" library_urn="urn:adsk.eagle:library:371" deviceset="GND" device=""/>
+<part name="C19" library="rcl" library_urn="urn:adsk.eagle:library:334" deviceset="C-EU" device="025-024X044" package3d_urn="urn:adsk.eagle:package:23630/1" value="0.1u"/>
 </parts>
 <sheets>
@@
 <instance part="GND14" gate="1" x="64.77" y="12.7" smashed="yes" rot="R90">
 <attribute name="VALUE" x="67.31" y="10.16" size="1.778" layer="96" rot="R90"/>
+</instance>
+<instance part="GND19" gate="1" x="71.12" y="15.24" smashed="yes" rot="R90">
+<attribute name="VALUE" x="73.66" y="12.7" size="1.778" layer="96" rot="R90"/>
+</instance>
+<instance part="C19" gate="G$1" x="64.77" y="25.4" smashed="yes" rot="R90">
+<attribute name="NAME" x="64.389" y="26.924" size="1.778" layer="95" rot="R90"/>
+<attribute name="VALUE" x="69.469" y="26.924" size="1.778" layer="96" rot="R90"/>
 </instance>
 </instances>
@@
 <pinref part="GND14" gate="1" pin="GND"/>
 <pinref part="SV1" gate="1" pin="1"/>
+</segment>
+<segment>
+<pinref part="SV1" gate="1" pin="2"/>
+<wire x1="62.23" y1="15.24" x2="68.58" y2="15.24" width="0.1524" layer="91"/>
+<pinref part="GND19" gate="1" pin="GND"/>
 </segment>
 </net>
@@
 </segment>
 </net>
-<net name="N$8" class="0">
+<net name="RESET" class="0">
 <segment>
 <pinref part="R9" gate="G$1" pin="2"/>
 <pinref part="U1" gate="G$1" pin="PC6(/RESET)"/>
 <wire x1="6.35" y1="142.24" x2="8.89" y2="142.24" width="0.1524" layer="91"/>
+<label x="5.08" y="143.51" size="1.778" layer="95"/>
+</segment>
+<segment>
+<pinref part="C19" gate="G$1" pin="2"/>
+<wire x1="69.85" y1="25.4" x2="72.39" y2="25.4" width="0.1524" layer="91"/>
+<label x="71.12" y="25.4" size="1.778" layer="95"/>
 </segment>
 </net>
@@
 <label x="-53.34" y="111.76" size="1.778" layer="95"/>
 </segment>
+<segment>
+<pinref part="SV1" gate="1" pin="5"/>
+<wire x1="62.23" y1="22.86" x2="63.5" y2="22.86" width="0.1524" layer="91"/>
+<label x="63.5" y="22.86" size="1.778" layer="95"/>
+</segment>
 </net>
 <net name="PADRIN" class="0">
@@
 </segment>
 </net>
+<net name="RX" class="0">
+<segment>
+<pinref part="SV1" gate="1" pin="4"/>
+<wire x1="62.23" y1="20.32" x2="63.5" y2="20.32" width="0.1524" layer="91"/>
+<label x="63.5" y="20.32" size="1.778" layer="95"/>
+</segment>
+<segment>
+<pinref part="U1" gate="G$1" pin="PD0(RXD)"/>
+<wire x1="57.15" y1="119.38" x2="59.69" y2="119.38" width="0.1524" layer="91"/>
+<label x="59.69" y="119.38" size="1.778" layer="95"/>
+</segment>
+</net>
+<net name="N$6" class="0">
+<segment>
+<pinref part="C19" gate="G$1" pin="1"/>
+<pinref part="SV1" gate="1" pin="6"/>
+</segment>
+</net>

Commit message: changed pad
Connections:
- net BUZ+: now also U1.PD5(T1); no longer U1.PC0(ADC0)
- net PADLIN: now also U1.PC0(ADC0); no longer U1.PC2(ADC2)
- net PADR: now also U1.PC2(ADC2); no longer U1.PD2(INT0)
Changed lines of the file:
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@@
 </segment>
 <segment>
-<pinref part="U1" gate="G$1" pin="PC0(ADC0)"/>
-<wire x1="57.15" y1="142.24" x2="59.69" y2="142.24" width="0.1524" layer="91"/>
-<label x="59.69" y="142.24" size="1.778" layer="95"/>
+<pinref part="U1" gate="G$1" pin="PD5(T1)"/>
+<wire x1="57.15" y1="106.68" x2="59.69" y2="106.68" width="0.1524" layer="91"/>
+<label x="59.69" y="106.68" size="1.778" layer="95"/>
 </segment>
 </net>
@@
 <net name="PADR" class="0">
 <segment>
-<pinref part="U1" gate="G$1" pin="PD2(INT0)"/>
-<wire x1="57.15" y1="114.3" x2="59.69" y2="114.3" width="0.1524" layer="91"/>
-<label x="59.69" y="114.3" size="1.778" layer="95"/>
-</segment>
-<segment>
 <label x="114.3" y="53.34" size="1.778" layer="95"/>
 <pinref part="PIN2" gate="G$1" pin="P$1"/>
@@
 <wire x1="97.79" y1="53.34" x2="99.06" y2="53.34" width="0.1524" layer="91"/>
 <junction x="97.79" y="53.34"/>
+</segment>
+<segment>
+<pinref part="U1" gate="G$1" pin="PC2(ADC2)"/>
+<wire x1="57.15" y1="137.16" x2="58.42" y2="137.16" width="0.1524" layer="91"/>
+<label x="58.42" y="137.16" size="1.778" layer="95"/>
 </segment>
 </net>
@@
 </segment>
 <segment>
-<pinref part="U1" gate="G$1" pin="PC2(ADC2)"/>
-<wire x1="57.15" y1="137.16" x2="58.42" y2="137.16" width="0.1524" layer="91"/>
-<label x="58.42" y="137.16" size="1.778" layer="95"/>
-</segment>
-</net>
+<pinref part="U1" gate="G$1" pin="PC0(ADC0)"/>
+<wire x1="57.15" y1="142.24" x2="59.69" y2="142.24" width="0.1524" layer="91"/>
+<label x="59.69" y="142.24" size="1.778" layer="95"/>
+</segment>
+</net>
